File: pcb/manipulation.kicad_sch (KiCad schematic)
At the start: 11 parts, among them M5 Corkscrew, M6 Crank, M7 Fingers, U12 TB9051FTG, U13 TB9051FTG, U7 DRV8833, U8 DRV8833

Commit message: Fix ERC issues and layout connectors
Parts:
- renumbered M7 to M5, M5 to M6, M6 to M7, U7 to U11, U8 to U12, U12 to U13, U13 to U14
Connections:
- net CORKSCREW_PWM1: now also U13.8 (PWM1)
- net CORKSCREW_PWM2: now also U13.7 (PWM2)
- net CRANK_PWM1: now also U14.8 (PWM1)
- net CRANK_PWM2: now also U14.7 (PWM2)
- net F3_PWM1: now also U12.7 (IN1)
- net F3_PWM2: now also U12.8 (IN2)
- net F4_PWM1: now also U12.11 (IN3)
- net F4_PWM2: now also U12.12 (IN4)

Commit message: Route I2C and planes
Connections:
- net CORKSCREW_OUT1: now also U13.11 (OUT1); no longer U13.12 (OUT2)
- net CORKSCREW_OUT2: now also U13.12 (OUT2); no longer U13.11 (OUT1)
Changed lines of the file:
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@@
 		)
 	)
-	(label "CORKSCREW_OUT2"
+	(label "CORKSCREW_OUT1"
 		(at 160.02 44.45 0)
 		(effects
@@
 		)
 	)
-	(label "CORKSCREW_OUT1"
+	(label "CORKSCREW_OUT2"
 		(at 160.02 40.64 0)
 		(effects
