File: pcb/ieee.kicad_pcb (KiCad board)
At the start: 4 copper layers, 152.4 x 114.3 mm, 47 parts, among them J1 Screw_Terminal_01x02, J2 Conn_01x20_Pin, J3 Conn_01x20_Pin, J4 I2C_LCD, J5 Conn_01x20_Pin, J6 Conn_01x20_Pin, M1 FL, M2 RL, M3 FR, M4 RR, M5 Fingers, M6 Corkscrew, M7 Crank, SW1 SW_SPST, U1 TCS34725, U10 TB9051FTG, U11 DRV8833, U12 DRV8833, U13 TB9051FTG, U14 TB9051FTG, U2 PCA9543AD_118, U3 D36V50F5, U4 TCS34725, U5 IR_Transmitter, U6 SN74LVC8T245NSR, U7 TB9051FTG, U8 TB9051FTG, U9 TB9051FTG

Commit message: Finish layout
Parts:
- removed the H2 at (242.3, 69.1)
- added C1: 0.1uF, Capacitor_SMD:C_0603_1608Metric_Pad1.08x0.95mm_HandSolder, F.Cu at (141.0, 108.5)
- added C2: 0.1uF, Capacitor_SMD:C_0603_1608Metric_Pad1.08x0.95mm_HandSolder, F.Cu at (144.6, 112.3)
- added C3: 0.1uF, Capacitor_SMD:C_0603_1608Metric_Pad1.08x0.95mm_HandSolder, F.Cu at (152.1, 109.7)
- added C4: 0.1uF, Capacitor_SMD:C_0603_1608Metric_Pad1.08x0.95mm_HandSolder, F.Cu at (162.8, 48.0)
- added C5: 0.1uF, Capacitor_SMD:C_0603_1608Metric_Pad1.08x0.95mm_HandSolder, F.Cu at (130.8, 40.1)
- added C6: 0.1uF, Capacitor_SMD:C_0603_1608Metric_Pad1.08x0.95mm_HandSolder, F.Cu at (169.2, 41.4)
- added C7: 0.1uF, Capacitor_SMD:C_0603_1608Metric_Pad1.08x0.95mm_HandSolder, F.Cu at (176.7, 49.5)
- added C8: 1uF, Capacitor_SMD:C_0603_1608Metric_Pad1.08x0.95mm_HandSolder, F.Cu at (165.7, 41.4)
- moved U10 13.3 mm to (108.2, 46.9)
- moved U7 13.3 mm to (108.2, 132.8)
- moved U8 13.3 mm to (108.2, 104.2)
- moved U9 13.3 mm to (108.2, 75.5)
- moved M1 13.3 mm to (89.4, 134.6)
- moved M2 13.3 mm to (89.4, 109.1)
- moved M3 13.3 mm to (89.4, 83.5)
- moved M4 13.3 mm to (89.4, 57.9)
- moved M6 13.3 mm to (159.6, 145.0)
- moved M7 13.3 mm to (130.3, 144.8)
- moved U13 13.3 mm to (166.4, 129.3)
- moved U14 13.3 mm to (135.7, 129.3)
- moved H2 12.7 mm to (88.9, 38.1)
- moved H3 12.7 mm to (88.9, 142.2)
- moved J1 7.65 mm to (216.4, 130.3)
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- renumbered H3 to H2, H4 to H3
Connections:
- A3 pad 10: /pico_subsystem/RL_PWM1 -> /pico_subsystem/RL_PWM2
- A3 pad 11: /pico_subsystem/PICO_GPIO8 -> /pico_subsystem/FL_PWM1
- A3 pad 12: /pico_subsystem/PICO_GPIO9 -> /pico_subsystem/FL_PWM2
- A3 pad 21: /pico_subsystem/RR_PWM1 -> /pico_subsystem/PICO_GPIO16
- A3 pad 22: /pico_subsystem/RR_PWM2 -> /pico_subsystem/PICO_GPIO17
- A3 pad 4: /pico_subsystem/FL_PWM2 -> /pico_subsystem/RR_PWM1
- A3 pad 5: /pico_subsystem/FL_PWM1 -> /pico_subsystem/RR_PWM2
- A3 pad 6: /pico_subsystem/FR_PWM2 -> /pico_subsystem/FR_PWM1
- A3 pad 7: /pico_subsystem/FR_PWM1 -> /pico_subsystem/FR_PWM2
- A3 pad 9: /pico_subsystem/RL_PWM2 -> /pico_subsystem/RL_PWM1
- J5 pad 10: /pico_subsystem/RL_PWM1 -> /pico_subsystem/RL_PWM2
- J5 pad 11: /pico_subsystem/PICO_GPIO8 -> /pico_subsystem/FL_PWM1
- J5 pad 12: /pico_subsystem/PICO_GPIO9 -> /pico_subsystem/FL_PWM2
- J5 pad 4: /pico_subsystem/FL_PWM2 -> /pico_subsystem/RR_PWM1
- J5 pad 5: /pico_subsystem/FL_PWM1 -> /pico_subsystem/RR_PWM2
- J5 pad 6: /pico_subsystem/FR_PWM2 -> /pico_subsystem/FR_PWM1
- J5 pad 7: /pico_subsystem/FR_PWM1 -> /pico_subsystem/FR_PWM2
- J5 pad 9: /pico_subsystem/RL_PWM2 -> /pico_subsystem/RL_PWM1
- J6 pad 19: /pico_subsystem/RR_PWM2 -> /pico_subsystem/PICO_GPIO17
- J6 pad 20: /pico_subsystem/RR_PWM1 -> /pico_subsystem/PICO_GPIO16
- JP1 pad 1: /manipulation/CRANK_PWM1 -> /manipulation/CRANK_PWM2
- JP2 pad 1: /manipulation/CRANK_PWM2 -> /manipulation/CRANK_PWM1
- JP3 pad 1: /manipulation/CRANK_PWM1 -> /manipulation/CRANK_PWM2
- JP4 pad 1: /manipulation/CRANK_PWM2 -> /manipulation/CRANK_PWM1
- SW1 pad 1: /RPI_GPIO26 -> /RPI_GPIO21
- U1 pad 1: /RPI_GPIO21 -> /RPI_GPIO4
- U11 pad 11: /RPI_GPIO6 -> /RPI_GPIO16
- U11 pad 12: /RPI_GPIO7 -> /RPI_GPIO26
- U11 pad 7: /RPI_GPIO4 -> /RPI_GPIO5
- U11 pad 8: /RPI_GPIO5 -> /RPI_GPIO6
- U12 pad 11: /RPI_GPIO10 -> /RPI_GPIO9
- U12 pad 12: /RPI_GPIO11 -> /RPI_GPIO10
- U12 pad 8: /RPI_GPIO9 -> /RPI_GPIO11
- U13 pad 7: /RPI_GPIO17 -> /RPI_GPIO22
- U13 pad 8: /RPI_GPIO16 -> /RPI_GPIO23
- U2 pad 11: /RPI_GPIO22 -> /RPI_GPIO17
- U4 pad 1: /RPI_GPIO21 -> /RPI_GPIO4
- U5 pad 3: /pico_subsystem/PICO_GPIO15 -> /pico_subsystem/PICO_GPIO10
- U6 pad 16: /pico_subsystem/RL_ENCB_5V -> /pico_subsystem/FR_ENCB_5V
- U6 pad 17: /pico_subsystem/RL_ENCA_5V -> /pico_subsystem/FR_ENCA_5V
- U6 pad 18: /pico_subsystem/FR_ENCB_5V -> /pico_subsystem/RL_ENCB_5V
- U6 pad 19: /pico_subsystem/FR_ENCA_5V -> /pico_subsystem/RL_ENCA_5V
Routing:
- net /manipulation/CRANK_PWM2: track 2.54 -> 138.7 mm
- net /manipulation/CRANK_PWM1: track 2.54 -> 138.5 mm
- net /pico_subsystem/PICO_3V3: track 5.08 -> 118.5 mm
- net /RPI_PWM0: track 6.10 -> 110.4 mm, vias 0 -> 1
- net /RPI_PWM1: track 12.2 -> 112.5 mm, vias 0 -> 1
- net /RPI_GPIO23: track 6.10 -> 91.3 mm, vias 0 -> 1
- net /pico_subsystem/RR_ENCB_5V: track 0.00 -> 83.4 mm
- net /pico_subsystem/RR_ENCA_5V: track 0.00 -> 82.7 mm
- net /RPI_GPIO22: track 12.2 -> 93.8 mm, vias 0 -> 1
- net /RPI_GPIO21: track 11.2 -> 88.1 mm
- net /pico_subsystem/RL_ENCB_5V: track 0.00 -> 75.3 mm
- net /pico_subsystem/RL_ENCA_5V: track 0.00 -> 73.0 mm
- net /pico_subsystem/FR_ENCB_5V: track 0.00 -> 67.8 mm
- net /pico_subsystem/FR_ENCA_5V: track 0.00 -> 66.1 mm
- net /pico_subsystem/FL_PWM2: track 5.08 -> 67.2 mm
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Other:
- board size 152.4 x 114.3 mm -> 139.7 x 114.3 mm
